Commit message: update urdf export

File: mechanical/Simulation Files/ava2/urdf/ava2.urdf (robot description, URDF)
Before this commit: robot FullAssembly_AVA_2_0.SLDASM, 26 links, 25 joints
Links:
- link abdominals: mass 0.353477688972343 -> 0.353477688976877
- link bicep_left: mass 0.232287327837173 -> 0.232287327840107
- link chest: mass 0.756245533149595 -> 0.756245533173823
- link foot_left: mass 0.0853987779456411 -> 0.0853987779456404
- link foot_right: mass 0.0853737511932979 -> 0.0853737511932987
- link forearm_left: mass 0.0700934249374858 -> 0.0700934249374856
- link hand_left: mass 0.0198788406763806 -> 0.019878840672065
- link hand_right: mass 0.0198788582866051 -> 0.0198788582824736
- link head: mass 0.366246371096136 -> 0.366246371096135
- link hip_left: mass 0.178323461769503 -> 0.178323461736544
- link hip_right: mass 0.178325355978329 -> 0.178325355992848
- link hipconnector_left: mass 0.169598324220792 -> 0.169598324229684
- link hipconnector_right: mass 0.169598376951876 -> 0.169598376961271
- link pelvis: mass 0.351826948016737 -> 0.351826948011236
- link shoulder_left: mass 0.172050390082777 -> 0.17205039008692
- link shoulder_right: mass 0.0933140477910859 -> 0.0933140477887859
- link thigh_left: mass 0.373973684441803 -> 0.373973684430428
- link thigh_right: mass 0.373973704214647 -> 0.37397370421226
- link wrist_left: mass 0.0359196656987808 -> 0.0359196656987806
Joints:
- joint biceplift_left: origin xyz=-0.12 0.006 0.0485 rpy=0 0 3.1416 -> xyz=-0.12 0.006 0.0485 rpy=0 0 3.14159265358979
- joint biceplift_right: origin xyz=0 0.0302 0 rpy=0 -0.26691 3.1416 -> xyz=0 0.030199999999934 0 rpy=0 -0.266912354008724 3.14159265358979
- joint shoulderspin_left: origin xyz=0.2055 0.01858 -0.002605 rpy=3.1416 -1.5708 0 -> xyz=0.2055 0.01858 -0.002605 rpy=3.14159 -1.5708 0
- joint shoulderspin_right: origin xyz=-0.0269 0.01858 -0.002605 rpy=3.1459 -1.5708 0 -> xyz=-0.0269 0.01858 -0.002605 rpy=3.14159 -1.5708 0
