Commit message: fixed urdf mesh references for balancing/chess model

File: mechanical/cad/assemblies/ava2.0/Assems For URDF/Balancing_Chess_URDF/urdf/Balancing_Chess_URDF.urdf (robot description, URDF)
Before this commit: robot Balancing_Chess_URDF, 28 links, 27 joints
Links:
- link abdominalmotors: geometry collision mesh filename=../meshes/abdominalmotors.STL; visual mesh filename=../meshes/abdominalmotors.STL
- link bicep_left: geometry collision mesh filename=../meshes/bicep_left.STL; visual mesh filename=../meshes/bicep_left.STL
- link bicep_right: geometry collision mesh filename=../meshes/bicep_right.STL; visual mesh filename=../meshes/bicep_right.STL
- link calf_left: geometry collision mesh filename=../meshes/calf_left.STL; visual mesh filename=../meshes/calf_left.STL
- link calf_right: geometry collision mesh filename=../meshes/calf_right.STL; visual mesh filename=../meshes/calf_right.STL
- link chest: geometry collision mesh filename=../meshes/chest.STL; visual mesh filename=../meshes/chest.STL
- link elbow_left: geometry collision mesh filename=../meshes/elbow_left.STL; visual mesh filename=../meshes/elbow_left.STL
- link elbow_right: geometry collision mesh filename=../meshes/elbow_right.STL; visual mesh filename=../meshes/elbow_right.STL
- link foot_left: geometry collision mesh filename=../meshes/foot_left.STL; visual mesh filename=../meshes/foot_left.STL
- link foot_right: geometry collision mesh filename=../meshes/foot_right.STL; visual mesh filename=../meshes/foot_right.STL
- link forearm_left: geometry collision mesh filename=../meshes/forearm_left.STL; visual mesh filename=../meshes/forearm_left.STL
- link forearm_right: geometry collision mesh filename=../meshes/forearm_right.STL; visual mesh filename=../meshes/forearm_right.STL
- link gripper_left: geometry collision mesh filename=../meshes/gripper_left.STL; visual mesh filename=../meshes/gripper_left.STL
- link gripper_right: geometry collision mesh filename=../meshes/gripper_right.STL; visual mesh filename=../meshes/gripper_right.STL
- link hand_left: geometry collision mesh filename=../meshes/hand_left.STL; visual mesh filename=../meshes/hand_left.STL
- link hand_right: geometry collision mesh filename=../meshes/hand_right.STL; visual mesh filename=../meshes/hand_right.STL
- link head: geometry collision mesh filename=../meshes/head.STL; visual mesh filename=../meshes/head.STL
- link hiplift_left: geometry collision mesh filename=../meshes/hiplift_left.STL; visual mesh filename=../meshes/hiplift_left.STL
- link hiplift_right: geometry collision mesh filename=../meshes/hiplift_right.STL; visual mesh filename=../meshes/hiplift_right.STL
- link hiprotate_left: geometry collision mesh filename=../meshes/hiprotate_left.STL; visual mesh filename=../meshes/hiprotate_left.STL
- link hiprotate_right: geometry collision mesh filename=../meshes/hiprotate_right.STL; visual mesh filename=../meshes/hiprotate_right.STL
- link neck: geometry collision mesh filename=../meshes/neck.STL; visual mesh filename=../meshes/neck.STL
- link pelvis: geometry collision mesh filename=../meshes/pelvis.STL; visual mesh filename=../meshes/pelvis.STL
- link shoulder_left: geometry collision mesh filename=../meshes/shoulder_left.STL; visual mesh filename=../meshes/shoulder_left.STL
- link shoulder_right: geometry collision mesh filename=../meshes/shoulder_right.STL; visual mesh filename=../meshes/shoulder_right.STL
- link thigh_left: geometry collision mesh filename=../meshes/thigh_left.STL; visual mesh filename=../meshes/thigh_left.STL
- link thigh_right: geometry collision mesh filename=../meshes/thigh_right.STL; visual mesh filename=../meshes/thigh_right.STL
- link waist: geometry collision mesh filename=../meshes/waist.STL; visual mesh filename=../meshes/waist.STL
