Commit message: New URDF export in hopes meshes are fixed

File: mechanical/cad/assemblies/ava2.0/Assems For URDF/UpdatedBalancing_URDF/urdf/UpdatedBalancing_URDF.urdf (robot description, URDF)
Before this commit: robot UpdatedBalancing_URDF, 28 links, 27 joints
Links:
- link abdominals: geometry collision mesh filename=../meshes/abdominals.STL; visual mesh filename=../meshes/abdominals.STL
- link bicep_left: geometry collision mesh filename=../meshes/bicep_left.STL; visual mesh filename=../meshes/bicep_left.STL
- link bicep_right: geometry collision mesh filename=../meshes/bicep_right.STL; visual mesh filename=../meshes/bicep_right.STL
- link chest: geometry collision mesh filename=../meshes/chest.STL; visual mesh filename=../meshes/chest.STL
- link elbow_left: geometry collision mesh filename=../meshes/elbow_left.STL; visual mesh filename=../meshes/elbow_left.STL
- link elbow_right: geometry collision mesh filename=../meshes/elbow_right.STL; visual mesh filename=../meshes/elbow_right.STL
- link foot_left: geometry collision mesh filename=../meshes/foot_left.STL; visual mesh filename=../meshes/foot_left.STL
- link foot_right: geometry collision mesh filename=../meshes/foot_right.STL; visual mesh filename=../meshes/foot_right.STL
- link forearm_left: geometry collision mesh filename=../meshes/forearm_left.STL; visual mesh filename=../meshes/forearm_left.STL
- link forearm_right: geometry collision mesh filename=../meshes/forearm_right.STL; visual mesh filename=../meshes/forearm_right.STL
- link gripper_left: geometry collision mesh filename=../meshes/gripper_left.STL; visual mesh filename=../meshes/gripper_left.STL
- link gripper_right: geometry collision mesh filename=../meshes/gripper_right.STL; visual mesh filename=../meshes/gripper_right.STL
- link hand_left: geometry collision mesh filename=../meshes/hand_left.STL; visual mesh filename=../meshes/hand_left.STL
- link hand_right: geometry collision mesh filename=../meshes/hand_right.STL; visual mesh filename=../meshes/hand_right.STL
- link head: geometry collision mesh filename=../meshes/head.STL; visual mesh filename=../meshes/head.STL
- link hip_left: geometry collision mesh filename=../meshes/hip_left.STL; visual mesh filename=../meshes/hip_left.STL
- link hip_right: geometry collision mesh filename=../meshes/hip_right.STL; visual mesh filename=../meshes/hip_right.STL
- link hipconnector_left: geometry collision mesh filename=../meshes/hipconnector_left.STL; visual mesh filename=../meshes/hipconnector_left.STL
- link hipconnector_right: geometry collision mesh filename=../meshes/hipconnector_right.STL; visual mesh filename=../meshes/hipconnector_right.STL
- link neck: geometry collision mesh filename=../meshes/neck.STL; visual mesh filename=../meshes/neck.STL
- link pelvis: geometry collision mesh filename=../meshes/pelvis.STL; visual mesh filename=../meshes/pelvis.STL
- link shin_left: geometry collision mesh filename=../meshes/shin_left.STL; visual mesh filename=../meshes/shin_left.STL
- link shin_right: geometry collision mesh filename=../meshes/shin_right.STL; visual mesh filename=../meshes/shin_right.STL
- link shoulder_left: geometry collision mesh filename=../meshes/shoulder_left.STL; visual mesh filename=../meshes/shoulder_left.STL
- link shoulder_right: geometry collision mesh filename=../meshes/shoulder_right.STL; visual mesh filename=../meshes/shoulder_right.STL
- link thigh_left: geometry collision mesh filename=../meshes/thigh_left.STL; visual mesh filename=../meshes/thigh_left.STL
- link thigh_right: geometry collision mesh filename=../meshes/thigh_right.STL; visual mesh filename=../meshes/thigh_right.STL
- link waist: geometry collision mesh filename=../meshes/waist.STL; visual mesh filename=../meshes/waist.STL
